File: hardware/kicad/schematic/build_display/sheet_d_mcu.kicad_sch (KiCad schematic)
At the start: 5 parts

Commit message: cp3: fplib footprint-dims inventory + fab-drill scan; ESP32 module HSvia0.3 variant (stock 0.2mm EP vias violate JLCPCB 0.3mm floor) — both boards, gates green
Co-Authored-By: Claude Fable 5 <noreply@anthropic.com>
Claude-Session: https://claude.ai/code/session_01EP34oLvQKnuhf59mAfUYQf
Parts:
- MOD1: footprint RF_Module:ESP32-S3-WROOM-1 -> volthium:ESP32-S3-WROOM-1_HSvia0.3
Changed lines of the file:
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@@
       (effects (font (size 1.0 1.0)) (justify left))
     )
-    (property "Footprint" "RF_Module:ESP32-S3-WROOM-1" (at 144.78 105.41 0)
+    (property "Footprint" "volthium:ESP32-S3-WROOM-1_HSvia0.3" (at 144.78 105.41 0)
       (effects (font (size 1.0 1.0)) hide)
     )
@@
     (instances
       (project "volthium_display"
-        (path "/c0199742-5bcb-45bb-97cf-4571618f61b3/8f61eaf4-748f-4563-87a1-b3a18dfc7cd1"
+        (path "/5acc4b28-7967-4916-84f2-72575ad52558/5d6a0f5f-9333-4ba6-9be2-333de371d4e3"
           (reference "MOD1") (unit 1)
         )
@@
     (instances
       (project "volthium_display"
-        (path "/c0199742-5bcb-45bb-97cf-4571618f61b3/8f61eaf4-748f-4563-87a1-b3a18dfc7cd1"
+        (path "/5acc4b28-7967-4916-84f2-72575ad52558/5d6a0f5f-9333-4ba6-9be2-333de371d4e3"
           (reference "C3") (unit 1)
         )
@@
     (instances
       (project "volthium_display"
-        (path "/c0199742-5bcb-45bb-97cf-4571618f61b3/8f61eaf4-748f-4563-87a1-b3a18dfc7cd1"
+        (path "/5acc4b28-7967-4916-84f2-72575ad52558/5d6a0f5f-9333-4ba6-9be2-333de371d4e3"
           (reference "C4") (unit 1)
         )
@@
     (instances
       (project "volthium_display"
-        (path "/c0199742-5bcb-45bb-97cf-4571618f61b3/8f61eaf4-748f-4563-87a1-b3a18dfc7cd1"
+        (path "/5acc4b28-7967-4916-84f2-72575ad52558/5d6a0f5f-9333-4ba6-9be2-333de371d4e3"
           (reference "R1") (unit 1)
         )
@@
     (instances
       (project "volthium_display"
-        (path "/c0199742-5bcb-45bb-97cf-4571618f61b3/8f61eaf4-748f-4563-87a1-b3a18dfc7cd1"
+        (path "/5acc4b28-7967-4916-84f2-72575ad52558/5d6a0f5f-9333-4ba6-9be2-333de371d4e3"
           (reference "C5") (unit 1)
         )
@@
   )
   (sheet_instances
-    (path "/c0199742-5bcb-45bb-97cf-4571618f61b3/8f61eaf4-748f-4563-87a1-b3a18dfc7cd1" (page "5"))
+    (path "/5acc4b28-7967-4916-84f2-72575ad52558/5d6a0f5f-9333-4ba6-9be2-333de371d4e3" (page "5"))
   )
 )
