File: hardware/kicad/schematic/build_display/sheet_d_mcu.kicad_sch (KiCad schematic)
At the start: 5 parts

Commit message: CP3: battery-side placement (#14)
* cp3: retire pass-1 PCB toolchain to archive/pass1_pcb; refresh kicad README + audit-tool defaults; prune dead .gitignore paths

Co-Authored-By: Claude Fable 5 <noreply@anthropic.com>
Claude-Session: https://claude.ai/code/session_01EP34oLvQKnuhf59mAfUYQf

* cp3: fplib footprint-dims inventory + fab-drill scan; ESP32 module HSvia0.3 variant (stock 0.2mm EP vias violate JLCPCB 0.3mm floor) — both boards, gates green

Co-Authored-By: Claude Fable 5 <noreply@anthropic.com>
Claude-Session: https://claude.ai/code/session_01EP34oLvQKnuhf59mAfUYQf

* cp3: battery placement generator green — 123 parts placed, analytic gates + strict DRC clean

pcb/core.py: netlist-parity/courtyard/outline/fab-rule/readback gates,
transactional DRC+renders, build-start poisons, refdes auto-placer,
kiutils KiCad-10 repairs (pad-angle composition, remove_unused_layers
inversion, property-block restoration). pcb/build.py: full battery-side
floorplan as data with probed connector orientations.

Co-Authored-By: Claude Fable 5 <noreply@anthropic.com>
Claude-Session: https://claude.ai/code/session_01EP34oLvQKnuhf59mAfUYQf

* cp3: visual-review fixes — ADM2587E barrier axis rotated (logic N / iso S, probed + asserted), C12 at U7 VCC column, D2/C12 swap, on-body refdes deprioritized, mount-hole refs hidden

Co-Authored-By: Claude Fable 5 <noreply@anthropic.com>
Claude-Session: https://claude.ai/code/session_01EP34oLvQKnuhf59mAfUYQf

* cp3: iteration 1 handoff — packet + D38 + PR-8 fixes (U5/U6 flow orientation, iso cap rows under pins) + D11 evidence; semaphore -> reviewer_turn

Co-Authored-By: Claude Fable 5 <noreply@anthropic.com>
Claude-Session: https://claude.ai/code/session_01EP34oLvQKnuhf59mAfUYQf

* cp3: post-handoff adversarial self-review (packet 4.5) — silk floored at JLC 1.0/0.15 min with dense-row re-space to 0 silk findings, DRC-oracle refdes refine loop, D1/TVS1 current-path fix, Phoenix 1757242 header verified, honest packet claims

Co-Authored-By: Cl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
Parts:
- MOD1: footprint RF_Module:ESP32-S3-WROOM-1 -> volthium:ESP32-S3-WROOM-1_HSvia0.3
Changed lines of the file:
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@@
       (effects (font (size 1.0 1.0)) (justify left))
     )
-    (property "Footprint" "RF_Module:ESP32-S3-WROOM-1" (at 144.78 105.41 0)
+    (property "Footprint" "volthium:ESP32-S3-WROOM-1_HSvia0.3" (at 144.78 105.41 0)
       (effects (font (size 1.0 1.0)) hide)
     )
@@
     (instances
       (project "volthium_display"
-        (path "/c0199742-5bcb-45bb-97cf-4571618f61b3/8f61eaf4-748f-4563-87a1-b3a18dfc7cd1"
+        (path "/5c155809-dc25-5751-9589-7c326e383180/9b37d860-4191-5f73-909b-625844c74c2a"
           (reference "MOD1") (unit 1)
         )
@@
     (instances
       (project "volthium_display"
-        (path "/c0199742-5bcb-45bb-97cf-4571618f61b3/8f61eaf4-748f-4563-87a1-b3a18dfc7cd1"
+        (path "/5c155809-dc25-5751-9589-7c326e383180/9b37d860-4191-5f73-909b-625844c74c2a"
           (reference "C3") (unit 1)
         )
@@
     (instances
       (project "volthium_display"
-        (path "/c0199742-5bcb-45bb-97cf-4571618f61b3/8f61eaf4-748f-4563-87a1-b3a18dfc7cd1"
+        (path "/5c155809-dc25-5751-9589-7c326e383180/9b37d860-4191-5f73-909b-625844c74c2a"
           (reference "C4") (unit 1)
         )
@@
     (instances
       (project "volthium_display"
-        (path "/c0199742-5bcb-45bb-97cf-4571618f61b3/8f61eaf4-748f-4563-87a1-b3a18dfc7cd1"
+        (path "/5c155809-dc25-5751-9589-7c326e383180/9b37d860-4191-5f73-909b-625844c74c2a"
           (reference "R1") (unit 1)
         )
@@
     (instances
       (project "volthium_display"
-        (path "/c0199742-5bcb-45bb-97cf-4571618f61b3/8f61eaf4-748f-4563-87a1-b3a18dfc7cd1"
+        (path "/5c155809-dc25-5751-9589-7c326e383180/9b37d860-4191-5f73-909b-625844c74c2a"
           (reference "C5") (unit 1)
         )
@@
   )
   (sheet_instances
-    (path "/c0199742-5bcb-45bb-97cf-4571618f61b3/8f61eaf4-748f-4563-87a1-b3a18dfc7cd1" (page "5"))
+    (path "/5c155809-dc25-5751-9589-7c326e383180/9b37d860-4191-5f73-909b-625844c74c2a" (page "5"))
   )
 )
