File: hardware/kicad/schematic/build_display/sheet_d_mcu.kicad_sch (KiCad schematic)
At the start: 5 parts

Commit message: cp4: open display placement — D39 decisions + two gate fixes found before placing
Pre-placement groundwork, all evidence-driven.

D39.1 MOD1 courtyard implements D26. The stock ESP32 courtyard is a T:
body stem plus a 48x21mm flare that exists ONLY to encode Espressif's
antenna keepout. D26 retired that keepout for this board (radio unused)
but the footprint never reflected it; honouring it would sterilise 36% of
an 85x65 PCB. New display-only variant _NoAntKeepout: 62/62 pads
coordinate-identical to the parent, sole graphic delta F.CrtYd 8 to 4
segments. Battery keeps the full-keepout parent (its radio IS used, D25).

D39.2 J2 is SIDE-entry (S8B), not top-entry (B8B). CP1 deferred this to
"CP3, from the depth stack" and it was never decided. JST ePH datasheet:
top-entry MATED height is 8.0mm (p.1), the entire PCB-to-module gap,
leaving nothing for the cable; side-entry is 7.6mm with the cable exiting
horizontally. Widening the gap is rejected by a coupling: plunger = gap +
faceplate + protrusion, so 8mm gives ~13.5mm (mid-catalog) but 12mm gives
~17.5mm (past catalog). Propagated to BOM, requirements, exact-part
contract, manifest key and the SUPERSEDED registry; the exact-part gate
caught the change en route.

GATE FIX 1 (latent, exposed by CP4's back-side parts): mounting holes were
registered on side F only, so a back-side part over a hole was invisible to
the side-aware collision gate. Now registered on both sides.

GATE FIX 2 (latent, worse): courtyard_segments handled only FpLine/FpRect
and silently skipped everything else, and a MountingHole courtyard is a
single fp_circle. Mounting holes have therefore contributed ZERO geometry
to the analytic gate all along; CP3's comment claiming they participate
like any part was false, and only DRC ever caught the hole-vs-jack overlap.
Now polygonalises circles (24 segments) and handles polys/arcs.
Poison-tested: part-on-hole fires on both sides; clear placement stays clean.

Regression check: the APPROVED battery board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
Parts:
- MOD1: footprint volthium:ESP32-S3-WROOM-1_HSvia0.3 -> volthium:ESP32-S3-WROOM-1_HSvia0.3_NoAntKeepout
Changed lines of the file:
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@@
       (effects (font (size 1.0 1.0)) (justify left))
     )
-    (property "Footprint" "volthium:ESP32-S3-WROOM-1_HSvia0.3" (at 144.78 105.41 0)
+    (property "Footprint" "volthium:ESP32-S3-WROOM-1_HSvia0.3_NoAntKeepout" (at 144.78 105.41 0)
       (effects (font (size 1.0 1.0)) hide)
     )
