File: hardware/kicad/schematic/build_display/sheet_d_power.kicad_sch (KiCad schematic)
At the start: 10 parts, among them U1 R-78E3.3-0.5, U3-LDO AP2112K-3.3, U4-MUX TPS2116DRLR

Commit message: cp2: display-iter1 findings F12-F15 resolved — responses in packet 9.5
F12: THVD1400 bus abs-max corrected to -16/+16 V (p.4) + operating
-7/+12 V (5.4), both re-derived from the on-file PDF (the first
correction attempt itself typed a recalled -14/+14 and was caught the
same way). F13: five SMD cells -> THT top-mount across cp1_bom /
cp1_battery_side / cp1_display_side / docs/hardware/bom; exact GCT
drawing fetched (browser-UA; sha 39afb82c5104), verified (Dip Type PCB
Top Mount, GF=Gold Flash, A=T&R), manifested as a distinct object with
the family-spec row demoted; doc_consistency gains an SMD-USB4085
rejection pattern (+3 fixtures, live-poison-proven) and an
[exact-object] drawing-coverage check. F14: bringup Stage 6 requires
display J5 fitted at the terminus + pre-attach J1 beep-out; new
display recovery appendix (J3 force-download, J-USB bench power, wake
triage) makes R18/R21 executable. F15: core readability gate now models
annotation-symbol VALUE text (reproduced all 4 reviewer defects before
the fix); flag blocks moved text above the glyph on BOTH boards incl.
the latent battery twin. Both builds green (display ERC rc=0/0 msgs,
battery rc=5/2-accepted), 42/42 requirements, label audit clean.
Semaphore -> reviewer_turn (display-iter2).

Co-Authored-By: Claude Fable 5 <noreply@anthropic.com>
Claude-Session: https://claude.ai/code/session_01EP34oLvQKnuhf59mAfUYQf
Changed lines of the file:
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@@
     (instances
       (project "volthium_display"
-        (path "/2949c5a9-47b5-4b33-9194-fa1ebcf4d0c4/ac0b2160-f7a4-4220-84cb-0eccd596ba64"
+        (path "/628936a5-da81-4c31-a24a-17c21b017a30/86bdac86-94a9-4145-97ab-c42fba98c28d"
           (reference "F1") (unit 1)
         )
@@
     (instances
       (project "volthium_display"
-        (path "/2949c5a9-47b5-4b33-9194-fa1ebcf4d0c4/ac0b2160-f7a4-4220-84cb-0eccd596ba64"
+        (path "/628936a5-da81-4c31-a24a-17c21b017a30/86bdac86-94a9-4145-97ab-c42fba98c28d"
           (reference "TVS1") (unit 1)
         )
@@
     (instances
       (project "volthium_display"
-        (path "/2949c5a9-47b5-4b33-9194-fa1ebcf4d0c4/ac0b2160-f7a4-4220-84cb-0eccd596ba64"
+        (path "/628936a5-da81-4c31-a24a-17c21b017a30/86bdac86-94a9-4145-97ab-c42fba98c28d"
           (reference "C1") (unit 1)
         )
@@
     (instances
       (project "volthium_display"
-        (path "/2949c5a9-47b5-4b33-9194-fa1ebcf4d0c4/ac0b2160-f7a4-4220-84cb-0eccd596ba64"
+        (path "/628936a5-da81-4c31-a24a-17c21b017a30/86bdac86-94a9-4145-97ab-c42fba98c28d"
           (reference "U1") (unit 1)
         )
@@
     (instances
       (project "volthium_display"
-        (path "/2949c5a9-47b5-4b33-9194-fa1ebcf4d0c4/ac0b2160-f7a4-4220-84cb-0eccd596ba64"
+        (path "/628936a5-da81-4c31-a24a-17c21b017a30/86bdac86-94a9-4145-97ab-c42fba98c28d"
           (reference "C2") (unit 1)
         )
@@
     (instances
       (project "volthium_display"
-        (path "/2949c5a9-47b5-4b33-9194-fa1ebcf4d0c4/ac0b2160-f7a4-4220-84cb-0eccd596ba64"
+        (path "/628936a5-da81-4c31-a24a-17c21b017a30/86bdac86-94a9-4145-97ab-c42fba98c28d"
           (reference "U3-LDO") (unit 1)
         )
@@
     (instances
       (project "volthium_display"
-        (path "/2949c5a9-47b5-4b33-9194-fa1ebcf4d0c4/ac0b2160-f7a4-4220-84cb-0eccd596ba64"
+        (path "/628936a5-da81-4c31-a24a-17c21b017a30/86bdac86-94a9-4145-97ab-c42fba98c28d"
           (reference "C_usb1") (unit 1)
         )
@@
     (instances
       (project "volthium_display"
-        (path "/2949c5a9-47b5-4b33-9194-fa1ebcf4d0c4/ac0b2160-f7a4-4220-84cb-0eccd596ba64"
+        (path "/628936a5-da81-4c31-a24a-17c21b017a30/86bdac86-94a9-4145-97ab-c42fba98c28d"
           (reference "U4-MUX") (unit 1)
         )
@@
     (instances
       (project "volthium_display"
-        (path "/2949c5a9-47b5-4b33-9194-fa1ebcf4d0c4/ac0b2160-f7a4-4220-84cb-0eccd596ba64"
+        (path "/628936a5-da81-4c31-a24a-17c21b017a30/86bdac86-94a9-4145-97ab-c42fba98c28d"
           (reference "C_usb2") (unit 1)
         )
@@
     (instances
       (project "volthium_display"
-        (path "/2949c5a9-47b5-4b33-9194-fa1ebcf4d0c4/ac0b2160-f7a4-4220-84cb-0eccd596ba64"
+        (path "/628936a5-da81-4c31-a24a-17c21b017a30/86bdac86-94a9-4145-97ab-c42fba98c28d"
           (reference "C_mux") (unit 1)
         )
@@
   (symbol (lib_id "volthium:PWR_FLAG") (at 185.42000000000002 129.54 0) (unit 1)
     (in_bom yes) (on_board yes)
-    (property "Reference" "#FLG1" (at 182.88 125.73 0)
-      (effects (font (size 1.0 1.0)) (justify left))
-    )
-    (property "Value" "PWR_FLAG" (at 181.61 133.35 0)
+    (property "Reference" "#FLG1" (at 182.88 123.19 0)
+      (effects (font (size 1.0 1.0)) (justify left))
+    )
+    (property "Value" "PWR_FLAG" (at 181.61 125.73 0)
       (effects (font (size 1.0 1.0)) (justify left))
     )
@@
     (instances
       (project "volthium_display"
-        (path "/2949c5a9-47b5-4b33-9194-fa1ebcf4d0c4/ac0b2160-f7a4-4220-84cb-0eccd596ba64"
+        (path "/628936a5-da81-4c31-a24a-17c21b017a30/86bdac86-94a9-4145-97ab-c42fba98c28d"
           (reference "#FLG1") (unit 1)
         )
@@
   (symbol (lib_id "volthium:PWR_FLAG") (at 203.2 129.54 0) (unit 1)
     (in_bom yes) (on_board yes)
-    (property "Reference" "#FLG2" (at 200.66 125.73 0)
-      (effects (font (size 1.0 1.0)) (justify left))
-    )
-    (property "Value" "PWR_FLAG" (at 199.39000000000001 133.35 0)
+    (property "Reference" "#FLG2" (at 200.66 123.19 0)
+      (effects (font (size 1.0 1.0)) (justify left))
+    )
+    (property "Value" "PWR_FLAG" (at 199.39000000000001 125.73 0)
       (effects (font (size 1.0 1.0)) (justify left))
     )
@@
     (instances
       (project "volthium_display"
-        (path "/2949c5a9-47b5-4b33-9194-fa1ebcf4d0c4/ac0b2160-f7a4-4220-84cb-0eccd596ba64"
+        (path "/628936a5-da81-4c31-a24a-17c21b017a30/86bdac86-94a9-4145-97ab-c42fba98c28d"
           (reference "#FLG2") (unit 1)
         )
@@
   (symbol (lib_id "volthium:PWR_FLAG") (at 220.98 129.54 0) (unit 1)
     (in_bom yes) (on_board yes)
-    (property "Reference" "#FLG3" (at 218.44 125.73 0)
-      (effects (font (size 1.0 1.0)) (justify left))
-    )
-    (property "Value" "PWR_FLAG" (at 217.17000000000002 133.35 0)
+    (property "Reference" "#FLG3" (at 218.44 123.19 0)
+      (effects (font (size 1.0 1.0)) (justify left))
+    )
+    (property "Value" "PWR_FLAG" (at 217.17000000000002 125.73 0)
       (effects (font (size 1.0 1.0)) (justify left))
     )
@@
     (instances
       (project "volthium_display"
-        (path "/2949c5a9-47b5-4b33-9194-fa1ebcf4d0c4/ac0b2160-f7a4-4220-84cb-0eccd596ba64"
+        (path "/628936a5-da81-4c31-a24a-17c21b017a30/86bdac86-94a9-4145-97ab-c42fba98c28d"
           (reference "#FLG3") (unit 1)
         )
@@
   (symbol (lib_id "volthium:PWR_FLAG") (at 238.76 129.54 0) (unit 1)
     (in_bom yes) (on_board yes)
-    (property "Reference" "#FLG4" (at 236.22 125.73 0)
-      (effects (font (size 1.0 1.0)) (justify left))
-    )
-    (property "Value" "PWR_FLAG" (at 234.95000000000002 133.35 0)
+    (property "Reference" "#FLG4" (at 236.22 123.19 0)
+      (effects (font (size 1.0 1.0)) (justify left))
+    )
+    (property "Value" "PWR_FLAG" (at 234.95000000000002 125.73 0)
       (effects (font (size 1.0 1.0)) (justify left))
     )
@@
     (instances
       (project "volthium_display"
-        (path "/2949c5a9-47b5-4b33-9194-fa1ebcf4d0c4/ac0b2160-f7a4-4220-84cb-0eccd596ba64"
+        (path "/628936a5-da81-4c31-a24a-17c21b017a30/86bdac86-94a9-4145-97ab-c42fba98c28d"
           (reference "#FLG4") (unit 1)
         )
@@
   )
   (sheet_instances
-    (path "/2949c5a9-47b5-4b33-9194-fa1ebcf4d0c4/ac0b2160-f7a4-4220-84cb-0eccd596ba64" (page "2"))
+    (path "/628936a5-da81-4c31-a24a-17c21b017a30/86bdac86-94a9-4145-97ab-c42fba98c28d" (page "2"))
   )
 )
