File: hardware/kicad/schematic/build_display/sheet_d_conn.kicad_sch (KiCad schematic)
At the start: 6 parts, among them J1 Wurth_615008145521, J3 ESP-Prog

Commit message: cp2: display-iter2 F16 resolved — render-calibrated glyph metrics + pdf-text ground-truth gate + SHIELD pin fix (packet 9.6)
Root cause: the glyph gate's assumed 0.85mm/char + 1.27mm text model
under-sized KiCad's real stroke-font rendering (fitz-measured 1.10-1.29
mm/char proportional, 1.91mm box height) and passed a real SHIELDxGND
ink collision on the shared USB_C_16P symbol. Fixes, gates-first: (1)
GLYPH_ADV/GLYPH_H render-calibrated constants with per-class thresholds
(text-text 0.3, text-art 0.7 -- art solids are outer hulls; clean
contacts measure to 0.59); (2) new [pdf-text] gate in render() checking
the exported PDF's deduplicated word boxes at 0.5mm (calibrated between
the reviewer-eye-cleared 0.42 box contact and the 0.64 real ink
overlap) -- the reviewer's second-opinion script as a standing gate;
both proven by rebuilding the unfixed symbol: exactly 2 SHIELDxGND
failures per board, nothing else. (3) volthium.kicad_sym SH pin -15.24
-> -12.7 (SBU2 row); fitz re-measures zero intersections. Both boards
green (display ERC rc=0, battery rc=5/2-accepted), 42/42, label audit
+ doc consistency clean. kicad skill v0.2.2 (separate repo) carries
the distilled lesson; codex's popup-preflight branch merged as v0.2.1.

Co-Authored-By: Claude Fable 5 <noreply@anthropic.com>
Claude-Session: https://claude.ai/code/session_01EP34oLvQKnuhf59mAfUYQf
Changed lines of the file:
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@@
     (stroke (width 0.1524) (type default))
   )
-  (wire (pts (xy 49.53 134.62) (xy 41.910000000000004 134.62))
+  (wire (pts (xy 49.53 132.08) (xy 41.910000000000004 132.08))
     (stroke (width 0.1524) (type default))
   )
@@
     (effects (font (size 1.0 1.0)) (justify right))
   )
-  (global_label "GND" (shape input) (at 41.910000000000004 134.62 0) (fields_autoplaced)
+  (global_label "GND" (shape input) (at 41.910000000000004 132.08 0) (fields_autoplaced)
     (effects (font (size 1.0 1.0)) (justify right))
   )
@@
     (instances
       (project "volthium_display"
-        (path "/628936a5-da81-4c31-a24a-17c21b017a30/3453d4f8-8ed0-4517-a76d-25092b74968d"
+        (path "/9ce06952-a670-413c-8891-8620b1692278/135787a8-c17e-4b1d-be1c-5648be200a0e"
           (reference "J1") (unit 1)
         )
@@
     (instances
       (project "volthium_display"
-        (path "/628936a5-da81-4c31-a24a-17c21b017a30/3453d4f8-8ed0-4517-a76d-25092b74968d"
+        (path "/9ce06952-a670-413c-8891-8620b1692278/135787a8-c17e-4b1d-be1c-5648be200a0e"
           (reference "J-USB") (unit 1)
         )
@@
     (instances
       (project "volthium_display"
-        (path "/628936a5-da81-4c31-a24a-17c21b017a30/3453d4f8-8ed0-4517-a76d-25092b74968d"
+        (path "/9ce06952-a670-413c-8891-8620b1692278/135787a8-c17e-4b1d-be1c-5648be200a0e"
           (reference "R_cc1") (unit 1)
         )
@@
     (instances
       (project "volthium_display"
-        (path "/628936a5-da81-4c31-a24a-17c21b017a30/3453d4f8-8ed0-4517-a76d-25092b74968d"
+        (path "/9ce06952-a670-413c-8891-8620b1692278/135787a8-c17e-4b1d-be1c-5648be200a0e"
           (reference "R_cc2") (unit 1)
         )
@@
     (instances
       (project "volthium_display"
-        (path "/628936a5-da81-4c31-a24a-17c21b017a30/3453d4f8-8ed0-4517-a76d-25092b74968d"
+        (path "/9ce06952-a670-413c-8891-8620b1692278/135787a8-c17e-4b1d-be1c-5648be200a0e"
           (reference "U-ESD") (unit 1)
         )
@@
     (instances
       (project "volthium_display"
-        (path "/628936a5-da81-4c31-a24a-17c21b017a30/3453d4f8-8ed0-4517-a76d-25092b74968d"
+        (path "/9ce06952-a670-413c-8891-8620b1692278/135787a8-c17e-4b1d-be1c-5648be200a0e"
           (reference "J3") (unit 1)
         )
@@
   )
   (sheet_instances
-    (path "/628936a5-da81-4c31-a24a-17c21b017a30/3453d4f8-8ed0-4517-a76d-25092b74968d" (page "3"))
+    (path "/9ce06952-a670-413c-8891-8620b1692278/135787a8-c17e-4b1d-be1c-5648be200a0e" (page "3"))
   )
 )

Commit message: cp4: D40 vertical USB-C (resolves DR-35) + D41 no signing keys (resolves DR-34)
D40 - the edge-mount USB4085 could not be plugged inside the wall box (~5mm
past any board edge vs a plug needing 15-20mm; popping the faceplate exposes
the board FRONT, not its edges). User chose the vertical option: it opens +Z
and is reachable straight-on once the faceplate and e-paper module come away,
and is invisible when assembled.

Part is GCT USB4115-03-C (9.30mm) rather than the shorter USB4120 (6.5mm),
deliberately trading depth for footprint provenance: KiCad ships a footprint
for the 4115 citing GCT's official drawing and none for the 4120, and
hand-authoring a 0.5mm-pitch connector land pattern is the exact risk class
that produced DR-33 and the CP3 mating-face defect. Depth is affordable here;
a wrong land pattern is not.

Checked rather than assumed: pin table cross-read against the drawing (the
footprint's A1-A12/B1-B12/SH pads are a superset of our 16-pin symbol, so
every pin binds and the 8 SuperSpeed pads float); 30/30 pad tuples identical
to the library so the lib_footprint_mismatch is the same serialisation class
(evidence in iter1/jusb_pad_diff.txt); nothing overhangs a board edge any
more, so the E-edge whitelist is gone and silk_edge_clearance went 2 -> 0.
I ALSO CORRECTED MYSELF: I had claimed the taller part would force a longer
button plunger. It does not - with the 15mm plunger already locked the
protrusion is 2.3mm, inside the 2-3mm spec. The arithmetic is in D40.

Depth stack re-driven: J-USB 9.30mm displaces J3's 9.1mm, so gap ~9.7mm and
stack ~34.7mm against ~45mm usable. Battery board KEEPS USB4085 - it is not
in a wall box and its edge mount is correct there.

D41 - RPA sign-off stays name-based (git authorship), no signing keys. The
limit is stated in the gate's docstring rather than papered over, and the
threat model in REVIEWER_PATCH_POLICY.md explains why it is proportionate.

Stale-claim sweep after the change: requirements.md's exact-part list sti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
Parts:
- J-USB: value USB4085-GF-A -> USB4115-03-C; footprint Connector_USB:USB_C_Receptacle_GCT_USB4085 -> Connector_USB:USB_C_Receptacle_GCT_USB4115-03-C
Changed lines of the file:
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@@
       (effects (font (size 1.0 1.0)) (justify left))
     )
-    (property "Value" "USB4085-GF-A" (at 54.61 93.98 0)
+    (property "Value" "USB4115-03-C" (at 54.61 93.98 0)
       (effects (font (size 1.0 1.0)) (justify left))
     )
-    (property "Footprint" "Connector_USB:USB_C_Receptacle_GCT_USB4085" (at 59.69 119.38 0)
+    (property "Footprint" "Connector_USB:USB_C_Receptacle_GCT_USB4115-03-C" (at 59.69 119.38 0)
       (effects (font (size 1.0 1.0)) hide)
     )
