File: hardware/kicad/pcb/build/battery_pcb.kicad_pcb (KiCad board)
At the start: 2 copper layers, 100 x 80 mm, 127 parts, among them J1 Phoenix_MSTBA_2,5-2-G-5,08, J10 Amphenol_RJHSE-5380, J11 Amphenol_RJHSE-5380, J2 Amphenol_RJHSE-5380, J3 USB-C 2.0, J4 TERM, J5 ESP-Prog, J6 Amphenol_RJHSE-5380, J7 TERM, Q10 NTR4171P, Q11 NTR4171P, Q3 2N7002, Q4 2N7002, Q5 NTR4171P, U1 LM5166YDRCR, U10 ADM2587EBRWZ, U11 ADM2587EBRWZ, U2 R-78HB12-0.5, U3 THVD1400DR, U4 TPS3808G01DBVR, U5 AP2112K-3.3, U6 TPS2116DRLR, U7 TCAN332DR

Commit message: cp3: visual-review fixes — ADM2587E barrier axis rotated (logic N / iso S, probed + asserted), C12 at U7 VCC column, D2/C12 swap, on-body refdes deprioritized, mount-hole refs hidden
Co-Authored-By: Claude Fable 5 <noreply@anthropic.com>
Claude-Session: https://claude.ai/code/session_01EP34oLvQKnuhf59mAfUYQf
Parts:
- moved C12 12.3 mm to (33.0, 56.0)
- moved D2 4.00 mm to (33.0, 60.0)
- turned U10 to 270 degrees
- turned U11 to 270 degrees
