File: hardware/kicad/pcb/build/battery_pcb.kicad_pcb (KiCad board)
At the start: 2 copper layers, 100 x 80 mm, 127 parts, among them J1 Phoenix_MSTBA_2,5-2-G-5,08, J10 Amphenol_RJHSE-5380, J11 Amphenol_RJHSE-5380, J2 Amphenol_RJHSE-5380, J3 USB-C 2.0, J4 TERM, J5 ESP-Prog, J6 Amphenol_RJHSE-5380, J7 TERM, Q10 NTR4171P, Q11 NTR4171P, Q3 2N7002, Q4 2N7002, Q5 NTR4171P, U1 LM5166YDRCR, U10 ADM2587EBRWZ, U11 ADM2587EBRWZ, U2 R-78HB12-0.5, U3 THVD1400DR, U4 TPS3808G01DBVR, U5 AP2112K-3.3, U6 TPS2116DRLR, U7 TCAN332DR

Commit message: wip: cp3 iter-2 fixes staged pre-handoff-check
Parts:
- moved L10 19.1 mm to (69.1, 62.0)
- moved L12 19.1 mm to (91.6, 62.0)
- moved L11 19.1 mm to (69.1, 58.2)
- moved L13 19.1 mm to (91.6, 58.2)
- moved R21 4.60 mm to (61.1, 35.6)
- moved R31 4.60 mm to (83.6, 35.6)
- moved R_byp2b 4.08 mm to (62.7, 24.6), turned to 90 degrees
- moved R22 2.00 mm to (51.1, 58.4)
- moved R23 2.00 mm to (51.1, 61.9)
- moved R32 2.00 mm to (73.6, 58.4)
- moved R33 2.00 mm to (73.6, 61.9)
