File: hardware/kicad/pcb/build_display/display_pcb.kicad_pcb (KiCad board)
At the start: 2 copper layers, 85 x 65 mm, 43 parts, among them J1 Wurth_615008145521, J2 JST_S8B-PH-K-S, J3 ESP-Prog, J5 TERM, U1 R-78E3.3-0.5, U2 THVD1400DR, U3-LDO AP2112K-3.3, U4-MUX TPS2116DRLR

Commit message: cp4: first fully gated display placement + DR-35 (USB-C access in the wall box)
All analytic gates and DRC pass: 43 footprints, 57 nets, accepted classes
only (unconnected 123 = placement-only; silk_edge_clearance 2 = designed
J-USB overhang; lib_footprint_mismatch 3 = vendored variants + flipped SIP,
per-instance evidence still owed in the packet).

Verified numerically after the mirror fix: U1 pads 27.41..32.48 sit inside
its B.CrtYd 24.13..35.85; J1 pads 2.05..17.55 inside 1.79..17.81. Back-side
geometry is now self-consistent.

DR-35 logged: the ordered USB-C is an EDGE connector, but the box leaves
only ~5mm beyond any board edge while a plug needs 15-20mm of approach, and
popping the faceplate exposes the board FRONT rather than its edges. Three
options costed; recommended accepting an unclip-to-service port. Must be
settled before CP6 exports the STEP the bracket is designed against.

Co-Authored-By: Claude Fable 5 <noreply@anthropic.com>
Claude-Session: https://claude.ai/code/session_01EP34oLvQKnuhf59mAfUYQf
Parts:
- moved J1 0.50 mm to (13.0, 28.8)
Changed lines of the file:
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@@
   )
   (footprint "volthium:J_Wurth_WR-MJ_615008145521" (version 20241229) (generator pcbnew) (layer "B.Cu")
-    (at 12.475000000000001 28.78 0)
+    (at 12.975000000000001 28.78 0)
     (descr "Modular Jack Horizontal Shielded w. EMI Panel Finger 8P8C CAT 5e Tab Down, body 15.8x21.14x19.1mm, https://www.we-online.com/en/components/products/datasheet/615008145521?ki")
     (tags "THT")

Commit message: cp4: correct the flip axis (mirror Y, not X) — KiCad's own library-match as oracle
My earlier flip fix mirrored the wrong axis. Settled empirically instead of
by reasoning: write a STOCK footprint to the back and let KiCad judge it.
lib_footprint_mismatch fires when a board footprint disagrees with its
library copy, so the correct transform is the one where a stock back-side
part reports NO mismatch.

  no mirror -> U1 mismatched
  mirror X  -> U1 mismatched  (my previous fix)
  mirror Y  -> U1 CLEAN

Corroborated against a shipped KiCad demo board: its B.Cu footprint stores
library-X with negated Y. Applied to both the writer (_flip_to_back) and the
gate transform (_xf) so they cannot diverge again; display
lib_footprint_mismatch dropped 3 -> 1 (only the vendored MOD1 variant, the
same kiutils-serialisation class CP3 accepted).

Placement re-fitted to the corrected back-side geometry: the 12 V + RS-485
front end moved into the clear y 6..25 band west of MOD1, since J1's pad
field now projects to x 6.9..25.4 / y 26.5..38.2.

Battery board re-verified byte-identical (448d59a276df) throughout.

DR-35 rewritten around the user's vertical-USB-C idea, which is better than
either option I had costed: GCT USB4120-03-C is 6.5mm tall (product spec p.1,
on file), the standoff gap is ~8mm and the tallest front part is already
~9.4mm, so it adds NO depth while making the port reachable straight-on with
the faceplate off. 89,250 in stock, /bin/zsh.84 CAD, Active, same vendor as the
incumbent. Recommended.

Skill: kicad v0.5.0 documents the whole double-sided workflow.

Co-Authored-By: Claude Fable 5 <noreply@anthropic.com>
Claude-Session: https://claude.ai/code/session_01EP34oLvQKnuhf59mAfUYQf
Parts:
- moved U2 24.1 mm to (12.5, 19.5)
- moved J5 10.0 mm to (28.0, 18.7)
- moved U1 10.0 mm to (24.5, 43.2)
- moved R2 8.54 mm to (21.5, 25.0)
- moved J1 8.50 mm to (13.0, 37.3)
- moved R3 7.91 mm to (21.5, 18.0)
- moved C1 6.52 mm to (12.5, 13.5)
- moved TVS2 6.52 mm to (23.5, 13.5)
- moved F1 6.08 mm to (10.5, 8.00)
- moved TVS1 6.02 mm to (23.5, 8.00)
- moved C8 6.00 mm to (10.0, 49.5)
- moved R4 5.41 mm to (27.0, 24.5)
- moved R5 4.00 mm to (16.0, 49.5)
